File: kicad-project-template.kicad_pcb (KiCad board)
At the start: 2 copper layers, 25.5 x 13.8 mm, 4 parts

Commit message: testing commit shorthash marking
Other:
- board size 25.5 x 13.8 mm -> 25.5 x 15 mm
- board text added: "${PROJECTNAME} ${BOARD_REV} ${BOARD_REV_DATE} ${PROJECT_GIT} ${GIT_SHORTHASH}"
- board text added: "${PROJECT_GIT} ${GIT_SHORTHASH}"
- board text removed: "${PROJECTNAME} ${BOARD_REV} ${BOARD_REV_DATE} ${PROJECT_GIT}"
- board text removed: "${PROJECT_GIT}"
Changed lines of the file:
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@@
 	(property "BOARD_REV" "1.0")
 	(property "BOARD_REV_DATE" "Feb 3 2025")
+	(property "GIT_SHORTHASH" "PLACEHOLDER")
 	(property "PROJECT_GIT" "github.com/tandej/kicad-project-template")
 	(property "SCH_REV" "1.0")
@@
 	(gr_rect
 		(start 138.75 96)
-		(end 164.25 109.75)
+		(end 164.25 111)
 		(stroke
 			(width 0.05)
@@
 		(layer "Edge.Cuts")
 	)
-	(gr_text "${PROJECTNAME}\n${BOARD_REV}\n${BOARD_REV_DATE}\n${PROJECT_GIT}"
-		(at 139 109.5 0)
+	(gr_text "${PROJECTNAME}\n${BOARD_REV}\n${BOARD_REV_DATE}\n${PROJECT_GIT}\n${GIT_SHORTHASH}"
+		(at 139 110.75 0)
 		(layer "F.SilkS")
 		(effects
@@
 		)
 	)
-	(gr_text "${PROJECT_GIT}"
+	(gr_text "${PROJECT_GIT}\n${GIT_SHORTHASH}"
 		(at 284.75 181.75 0)
 		(layer "Cmts.User")
@@
 	)
 	(gr_text "${AUTHOR}"
-		(at 285 183.5 0)
+		(at 284.75 184.5 0)
 		(layer "Cmts.User")
 		(effects
